File: Hardware/BTL_ESD/BTL_ESD.kicad_pcb (KiCad board)
At the start: 2 copper layers, 73.4 x 100 mm, 144 parts, among them J1 DC-005-5A-2.0, J2 Load Program, J3 Socket_TFT_1, J4 Socket_TFT_2, J5 USB_B_Micro, J6 220VAC, K1 SRD-05VDC-SL-C, Q1 MMBT2222A, Q2 MMBT2222A, Q3 MMBT2222A, Q4 MMBT2222A, SW1 MS-22D18G2ROHS, SW2 RESET, SW3 ENABLE, SW4 FLASH, U1 ICL7662CBA-T, U2 AMS1117-3.3, U3 TPS54331D, U4 STM32F103RCTx, U5 ESP32-WROOM-32E__4MB_HIGH_TEM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, U6 MCP6002-E_SN, U7 INA128UA, U8 CH340C, U9 PC817, Y1 8MHz, Y2 32.768KHz

Commit message: fea:STM32: upload structure fodler
Parts:
- removed H4: BoreHole, MountingHole:MountingHole_3.2mm_M3_Pad_TopBottom
- added J2: BOOT, Connector_PinHeader_2.54mm:PinHeader_1x03_P2.54mm_Vertical, F.Cu at (180.3, 69.2)
- added R15: Uart_Conn, UART:uart_conn, F.Cu at (185.3, 63.1)
- moved H3 208.5 mm to (222.8, 44.5)
- moved H2 180.8 mm to (222.1, 95.2)
- moved C23 164.6 mm to (200.8, 66.6), turned to 180 degrees
- moved C19 163.4 mm to (200.8, 68.6), turned to 180 degrees
- moved J3 147.4 mm to (201.7, 71.6), turned to -90 degrees
- moved C18 135.8 mm to (173.4, 70.0), turned to 180 degrees
- moved C17 135.6 mm to (173.4, 75.9), turned to 180 degrees
- moved R11 134.9 mm to (185.7, 69.2), turned to 180 degrees
- moved R12 134.9 mm to (185.7, 72.9)
- moved NT1 133.8 mm to (147.6, 91.4)
- moved C20 132.4 mm to (169.8, 71.5), turned to 90 degrees
- moved Y1 131.2 mm to (171.1, 80.0), turned to 180 degrees
- moved C21 127.6 mm to (165.4, 80.4), turned to 90 degrees
- moved Y2 127.1 mm to (173.0, 72.3)
- moved C22 124.8 mm to (162.6, 87.0), turned to -90 degrees
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- renumbered J2 to J3, J3 to J4, J4 to J5, J5 to J6, J6 to J7, R15 to R16, R16 to R17, R17 to R18, R18 to R19, R19 to R20, R20 to R21, R21 to R22, R22 to R23, R23 to R24, R24 to R25, R25 to R26, R26 to R27, R27 to R28, R28 to R29, R29 to R30, R30 to R31, R31 to R32
Connections:
- C41 pad 2: Flash -> FLASH
- D10 pad 1: V_USB -> D_P
- D10 pad 4: D_N -> V_USB
- D10 pad 6: D_P -> D_N
- R11 pad 2: /STM32/BOOT -> Net-(J2-Pin_1)
- R12 pad 1: /STM32/BOOT -> Net-(J2-Pin_3)
- R18 pad 2: Flash -> FLASH
- SW4 pad 1: Flash -> FLASH
- U4 pad 24: unconnected-(U4-PC4-Pad24) -> GPIO_1
- U4 pad 25: unconnected-(U4-PC5-Pad25) -> GPIO_2
- U4 pad 41: TFT_BL -> CONTROL_LED
- U4 pad 42: CONTROL_LED -> TFT_BL
- U4 pad 51: RXD -> UART4_TX
- U4 pad 52: TXD -> UART4_RX
- U5 pad 14: unconnected-(U5-IO12-Pad14) -> GPIO_1
- U5 pad 16: unconnected-(U5-IO13-Pad16) -> GPIO_2
- U5 pad 25: Flash -> FLASH
- U5 pad 27: RXD -> RXD_2
- U5 pad 28: TXD -> TXD_2
Routing:
- net +5V: track 35.2 -> 343.5 mm, vias 0 -> 17
- net +3V3: track 26.8 -> 270.4 mm, vias 0 -> 10
- net V_USB: track 3.20 -> 128.3 mm, vias 0 -> 8
- net EN: track 0.00 -> 104.8 mm, vias 0 -> 2
- net FLASH: track 0.00 -> 100.9 mm, vias 0 -> 4
- net TFT_IRQ: track 5.03 -> 78.6 mm, vias 1 -> 2
- net GPIO_1: track 0.00 -> 69.4 mm, vias 0 -> 2
- net SPI1_MISO: track 6.33 -> 75.7 mm
- net GPIO_2: track 0.00 -> 65.0 mm, vias 0 -> 2
- net SPI1_MOSI: track 0.00 -> 50.7 mm
- net CONTROL_LED: track 0.00 -> 49.3 mm, vias 0 -> 1
- net TFT_RESET: track 5.18 -> 53.5 mm, vias 1 -> 2
- net TFT_DC_RS: track 5.32 -> 52.8 mm, vias 1 -> 2
- net -5V: track 11.4 -> 55.9 mm, vias 0 -> 4
- net GND: track 46.5 -> 90.4 mm
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- added copper zone on B.Cu, net +3V3
- added copper zone on F.Cu, net +3V3
- added copper zone on B.Cu, net +5V
- added copper zone on F.Cu, net +5V
- added copper zone on F.Cu, net Net-(J7-Pin_1)
- added copper zone on B.Cu, net Net-(J7-Pin_4)
- added copper zone on B.Cu, net V_USB
- added copper zone on F.Cu, net V_USB
Other:
- board size 73.4 x 100 mm -> 73.4 x 95.8 mm

Commit message: update
Parts:
- moved TP1 12.0 mm to (131.0, 95.8)
- moved TP2 12.0 mm to (131.0, 100.4)
- moved TP3 12.0 mm to (131.0, 105.0)
- moved TP4 12.0 mm to (131.0, 109.6)
- moved H2 0.46 mm to (222.1, 95.7)
Routing:
- net /TFT/CONTROL_BL: track 10.9 -> 28.7 mm, vias 1 -> 2
- net TFT_BL: track 38.7 -> 34.8 mm
- net +5V: track 343.5 -> 340.7 mm
- net V_USB: track 128.3 -> 129.1 mm
