File: Hardware/BTL_ESD/BTL_ESD.kicad_sch (KiCad schematic)
At the start: 0 parts

Commit message: hardware: ver 1 schematic
Other:
- sheet TTL renamed USB_TTL
- sheet current_supply renamed CURRENT_SUPPLY
- sheet measure renamed MEASURE
- added sheet CONTROL_LED (control_led.kicad_sch)
- sheet USB_TTL: file TTL.kicad_sch -> USB_TTL.kicad_sch
Changed lines of the file:
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@@
     (stroke (width 0.1524) (type solid))
     (fill (color 0 0 0 0.0000))
-    (property "Sheetname" "TTL" (at 171.45 47.5484 0)
+    (property "Sheetname" "USB_TTL" (at 171.45 47.5484 0)
       (effects (font (size 1.27 1.27)) (justify left bottom))
     )
-    (property "Sheetfile" "TTL.kicad_sch" (at 171.45 78.0546 0)
+    (property "Sheetfile" "USB_TTL.kicad_sch" (at 171.45 78.0546 0)
       (effects (font (size 1.27 1.27)) (justify left top))
     )
@@
     (stroke (width 0.1524) (type solid))
     (fill (color 0 0 0 0.0000))
-    (property "Sheetname" "current_supply" (at 121.92 47.5484 0)
+    (property "Sheetname" "CURRENT_SUPPLY" (at 121.92 47.5484 0)
       (effects (font (size 1.27 1.27)) (justify left bottom))
     )
@@
     )
   )
+  (sheet (at 173.99 90.17) (size 29.21 26.67) (fields_autoplaced)
+    (stroke (width 0.1524) (type solid))
+    (fill (color 0 0 0 0.0000))
+    (property "Sheetname" "CONTROL_LED" (at 173.99 89.4584 0)
+      (effects (font (size 1.27 1.27)) (justify left bottom))
+    )
+    (property "Sheetfile" "control_led.kicad_sch" (at 173.99 117.4246 0)
+      (effects (font (size 1.27 1.27)) (justify left top))
+    )
+    (instances
+      (project "BTL_ESD"
+        (path "/ce4779b4-6d78-42e3-84df-0a4e77629b0f" (page "9"))
+      )
+    )
+  )
   (sheet (at 120.65 88.9) (size 34.29 27.94) (fields_autoplaced)
     (stroke (width 0.1524) (type solid))
     (fill (color 0 0 0 0.0000))
-    (property "Sheetname" "measure" (at 120.65 88.1884 0)
+    (property "Sheetname" "MEASURE" (at 120.65 88.1884 0)
       (effects (font (size 1.27 1.27)) (justify left bottom))
     )
