File: Hardware/BTL_ESD/USB_TTL.kicad_sch (KiCad schematic)
At the start: 14 parts, among them J5 USB_B_Micro, Q2 MMBT2222A, Q3 MMBT2222A, U8 CH340C

Commit message: update
Parts:
- renumbered D9 to D10, R25 to R26, R26 to R27, R27 to R28, R28 to R29
Changed lines of the file:
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@@
   (symbol (lib_id "power:GND") (at 82.55 115.57 0) (unit 1)
     (in_bom yes) (on_board yes) (dnp no) (fields_autoplaced)
-    (property "Reference" "#PWR071" (at 82.55 121.92 0)
+    (property "Reference" "#PWR074" (at 82.55 121.92 0)
       (effects (font (size 1.27 1.27)) hide)
     )
@@
       (project "BTL_ESD"
         (path "/ce4779b4-6d78-42e3-84df-0a4e77629b0f/5a62b24e-983b-422f-a5b4-3f2d2f2b7ed3"
-          (reference "#PWR071") (unit 1)
+          (reference "#PWR074") (unit 1)
         )
       )
@@
   (symbol (lib_id "power:GND") (at 154.94 73.66 0) (unit 1)
     (in_bom yes) (on_board yes) (dnp no) (fields_autoplaced)
-    (property "Reference" "#PWR074" (at 154.94 80.01 0)
+    (property "Reference" "#PWR077" (at 154.94 80.01 0)
       (effects (font (size 1.27 1.27)) hide)
     )
@@
       (project "BTL_ESD"
         (path "/ce4779b4-6d78-42e3-84df-0a4e77629b0f/5a62b24e-983b-422f-a5b4-3f2d2f2b7ed3"
-          (reference "#PWR074") (unit 1)
+          (reference "#PWR077") (unit 1)
         )
       )
@@
   (symbol (lib_id "Device:R_Small_US") (at 170.18 97.79 90) (unit 1)
     (in_bom yes) (on_board yes) (dnp no) (fields_autoplaced)
-    (property "Reference" "R25" (at 170.18 91.44 90)
+    (property "Reference" "R26" (at 170.18 91.44 90)
       (effects (font (size 1.27 1.27)))
     )
@@
       (project "BTL_ESD"
         (path "/ce4779b4-6d78-42e3-84df-0a4e77629b0f/5a62b24e-983b-422f-a5b4-3f2d2f2b7ed3"
-          (reference "R25") (unit 1)
+          (reference "R26") (unit 1)
         )
       )
@@
   (symbol (lib_id "SMF05C:SMF05C") (at 80.01 109.22 0) (unit 1)
     (in_bom yes) (on_board yes) (dnp no) (fields_autoplaced)
-    (property "Reference" "D9" (at 68.58 108.2357 0)
+    (property "Reference" "D10" (at 68.58 108.2357 0)
       (effects (font (size 1.27 1.27)) (justify right))
     )
@@
       (project "BTL_ESD"
         (path "/ce4779b4-6d78-42e3-84df-0a4e77629b0f/5a62b24e-983b-422f-a5b4-3f2d2f2b7ed3"
-          (reference "D9") (unit 1)
+          (reference "D10") (unit 1)
         )
       )
@@
   (symbol (lib_id "Device:R_US") (at 226.06 102.87 90) (unit 1)
     (in_bom yes) (on_board yes) (dnp no) (fields_autoplaced)
-    (property "Reference" "R28" (at 226.06 96.52 90)
+    (property "Reference" "R29" (at 226.06 96.52 90)
       (effects (font (size 1.27 1.27)))
     )
@@
       (project "BTL_ESD"
         (path "/ce4779b4-6d78-42e3-84df-0a4e77629b0f/5a62b24e-983b-422f-a5b4-3f2d2f2b7ed3"
-          (reference "R28") (unit 1)
+          (reference "R29") (unit 1)
         )
       )
@@
   (symbol (lib_id "power:GND") (at 57.15 102.87 0) (unit 1)
     (in_bom yes) (on_board yes) (dnp no) (fields_autoplaced)
-    (property "Reference" "#PWR070" (at 57.15 109.22 0)
+    (property "Reference" "#PWR073" (at 57.15 109.22 0)
       (effects (font (size 1.27 1.27)) hide)
     )
@@
       (project "BTL_ESD"
         (path "/ce4779b4-6d78-42e3-84df-0a4e77629b0f/5a62b24e-983b-422f-a5b4-3f2d2f2b7ed3"
-          (reference "#PWR070") (unit 1)
+          (reference "#PWR073") (unit 1)
         )
       )
@@
   (symbol (lib_id "power:GND") (at 147.32 113.03 0) (unit 1)
     (in_bom yes) (on_board yes) (dnp no) (fields_autoplaced)
-    (property "Reference" "#PWR073" (at 147.32 119.38 0)
+    (property "Reference" "#PWR076" (at 147.32 119.38 0)
       (effects (font (size 1.27 1.27)) hide)
     )
@@
       (project "BTL_ESD"
         (path "/ce4779b4-6d78-42e3-84df-0a4e77629b0f/5a62b24e-983b-422f-a5b4-3f2d2f2b7ed3"
-          (reference "#PWR073") (unit 1)
+          (reference "#PWR076") (unit 1)
         )
       )
@@
   (symbol (lib_id "Device:R_US") (at 226.06 77.47 90) (unit 1)
     (in_bom yes) (on_board yes) (dnp no) (fields_autoplaced)
-    (property "Reference" "R27" (at 226.06 71.12 90)
+    (property "Reference" "R28" (at 226.06 71.12 90)
       (effects (font (size 1.27 1.27)))
     )
@@
       (project "BTL_ESD"
         (path "/ce4779b4-6d78-42e3-84df-0a4e77629b0f/5a62b24e-983b-422f-a5b4-3f2d2f2b7ed3"
-          (reference "R27") (unit 1)
+          (reference "R28") (unit 1)
         )
       )
@@
   (symbol (lib_id "power:GND") (at 88.9 82.55 0) (unit 1)
     (in_bom yes) (on_board yes) (dnp no) (fields_autoplaced)
-    (property "Reference" "#PWR072" (at 88.9 88.9 0)
+    (property "Reference" "#PWR075" (at 88.9 88.9 0)
       (effects (font (size 1.27 1.27)) hide)
     )
@@
       (project "BTL_ESD"
         (path "/ce4779b4-6d78-42e3-84df-0a4e77629b0f/5a62b24e-983b-422f-a5b4-3f2d2f2b7ed3"
-          (reference "#PWR072") (unit 1)
+          (reference "#PWR075") (unit 1)
         )
       )
@@
   (symbol (lib_id "power:+5V") (at 187.96 62.23 0) (unit 1)
     (in_bom yes) (on_board yes) (dnp no) (fields_autoplaced)
-    (property "Reference" "#PWR075" (at 187.96 66.04 0)
+    (property "Reference" "#PWR078" (at 187.96 66.04 0)
       (effects (font (size 1.27 1.27)) hide)
     )
@@
       (project "BTL_ESD"
         (path "/ce4779b4-6d78-42e3-84df-0a4e77629b0f/5a62b24e-983b-422f-a5b4-3f2d2f2b7ed3"
-          (reference "#PWR075") (unit 1)
+          (reference "#PWR078") (unit 1)
         )
       )
@@
   (symbol (lib_id "power:GND") (at 187.96 77.47 0) (unit 1)
     (in_bom yes) (on_board yes) (dnp no) (fields_autoplaced)
-    (property "Reference" "#PWR076" (at 187.96 83.82 0)
+    (property "Reference" "#PWR079" (at 187.96 83.82 0)
       (effects (font (size 1.27 1.27)) hide)
     )
@@
       (project "BTL_ESD"
         (path "/ce4779b4-6d78-42e3-84df-0a4e77629b0f/5a62b24e-983b-422f-a5b4-3f2d2f2b7ed3"
-          (reference "#PWR076") (unit 1)
+          (reference "#PWR079") (unit 1)
         )
       )
@@
   (symbol (lib_id "Device:R_Small_US") (at 170.18 107.95 90) (unit 1)
     (in_bom yes) (on_board yes) (dnp no) (fields_autoplaced)
-    (property "Reference" "R26" (at 170.18 101.6 90)
+    (property "Reference" "R27" (at 170.18 101.6 90)
       (effects (font (size 1.27 1.27)))
     )
@@
       (project "BTL_ESD"
         (path "/ce4779b4-6d78-42e3-84df-0a4e77629b0f/5a62b24e-983b-422f-a5b4-3f2d2f2b7ed3"
-          (reference "R26") (unit 1)
-        )
-      )
+          (reference "R27") (unit 1)
+        )
+      )

Commit message: fea:STM32: upload structure fodler
Parts:
- renumbered J5 to J6, R26 to R27, R27 to R28, R28 to R29, R29 to R30
Connections:
- net D_N: now also D10.6; no longer D10.4
- net D_P: now also D10.1; no longer D10.6
- net V_USB: now also D10.4; no longer D10.1
Changed lines of the file:
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@@
   (junction (at 57.15 101.6) (diameter 0) (color 0 0 0 0)
   )
+  (junction (at 76.2 71.12) (diameter 0) (color 0 0 0 0)
+  )
+  (junction (at 72.39 90.17) (diameter 0) (color 0 0 0 0)
+  )
   (junction (at 218.44 102.87) (diameter 0) (color 0 0 0 0)
   )
-  (junction (at 92.71 90.17) (diameter 0) (color 0 0 0 0)
-  )
   (junction (at 187.96 74.93) (diameter 0) (color 0 0 0 0)
   )
-  (junction (at 72.39 71.12) (diameter 0) (color 0 0 0 0)
-  )
   (junction (at 218.44 77.47) (diameter 0) (color 0 0 0 0)
   )
+  (junction (at 85.09 92.71) (diameter 0) (color 0 0 0 0)
+  )
   (junction (at 81.28 71.12) (diameter 0) (color 0 0 0 0)
   )
   (junction (at 171.45 64.77) (diameter 0) (color 0 0 0 0)
-  )
-  (junction (at 82.55 92.71) (diameter 0) (color 0 0 0 0)
   )
   (junction (at 95.25 71.12) (diameter 0) (color 0 0 0 0)
@@
     (stroke (width 0) (type default))
   )
-  (wire (pts (xy 67.31 71.12) (xy 72.39 71.12))
+  (wire (pts (xy 92.71 100.33) (xy 85.09 100.33))
     (stroke (width 0) (type default))
   )
@@
     (stroke (width 0) (type default))
   )
-  (wire (pts (xy 82.55 92.71) (xy 86.36 92.71))
+  (wire (pts (xy 67.31 92.71) (xy 85.09 92.71))
     (stroke (width 0) (type default))
   )
@@
     (stroke (width 0) (type default))
   )
-  (wire (pts (xy 72.39 71.12) (xy 72.39 105.41))
-    (stroke (width 0) (type default))
-  )
   (wire (pts (xy 229.87 77.47) (xy 236.22 77.47))
     (stroke (width 0) (type default))
@@
     (stroke (width 0) (type default))
   )
+  (wire (pts (xy 92.71 105.41) (xy 92.71 100.33))
+    (stroke (width 0) (type default))
+  )
+  (wire (pts (xy 85.09 100.33) (xy 85.09 92.71))
+    (stroke (width 0) (type default))
+  )
   (wire (pts (xy 187.96 74.93) (xy 187.96 77.47))
     (stroke (width 0) (type default))
@@
     (stroke (width 0) (type default))
   )
+  (wire (pts (xy 72.39 90.17) (xy 99.06 90.17))
+    (stroke (width 0) (type default))
+  )
   (wire (pts (xy 154.94 66.04) (xy 154.94 67.31))
     (stroke (width 0) (type default))
@@
     (stroke (width 0) (type default))
   )
-  (wire (pts (xy 92.71 90.17) (xy 99.06 90.17))
-    (stroke (width 0) (type default))
-  )
   (wire (pts (xy 57.15 101.6) (xy 57.15 102.87))
     (stroke (width 0) (type default))
@@
     (stroke (width 0) (type default))
   )
-  (wire (pts (xy 82.55 92.71) (xy 82.55 105.41))
-    (stroke (width 0) (type default))
-  )
   (wire (pts (xy 218.44 86.36) (xy 243.84 93.98))
     (stroke (width 0) (type default))
@@
     (stroke (width 0) (type default))
   )
-  (wire (pts (xy 72.39 71.12) (xy 81.28 71.12))
+  (wire (pts (xy 67.31 71.12) (xy 76.2 71.12))
     (stroke (width 0) (type default))
   )
@@
     (stroke (width 0) (type default))
   )
+  (wire (pts (xy 82.55 105.41) (xy 82.55 85.09))
+    (stroke (width 0) (type default))
+  )
   (wire (pts (xy 163.83 104.14) (xy 163.83 107.95))
     (stroke (width 0) (type default))
@@
     (stroke (width 0) (type default))
   )
+  (wire (pts (xy 72.39 90.17) (xy 72.39 105.41))
+    (stroke (width 0) (type default))
+  )
+  (wire (pts (xy 76.2 71.12) (xy 81.28 71.12))
+    (stroke (width 0) (type default))
+  )
   (wire (pts (xy 171.45 64.77) (xy 171.45 67.31))
     (stroke (width 0) (type default))
   )
-  (wire (pts (xy 92.71 90.17) (xy 92.71 105.41))
-    (stroke (width 0) (type default))
-  )
   (wire (pts (xy 215.9 102.87) (xy 218.44 102.87))
     (stroke (width 0) (type default))
@@
     (stroke (width 0) (type default))
   )
+  (wire (pts (xy 85.09 92.71) (xy 86.36 92.71))
+    (stroke (width 0) (type default))
+  )
   (wire (pts (xy 171.45 72.39) (xy 171.45 74.93))
     (stroke (width 0) (type default))
@@
     (stroke (width 0) (type default))
   )
-  (wire (pts (xy 67.31 92.71) (xy 82.55 92.71))
+  (wire (pts (xy 82.55 85.09) (xy 76.2 85.09))
     (stroke (width 0) (type default))
   )
@@
     (stroke (width 0) (type default))
   )
-  (wire (pts (xy 67.31 90.17) (xy 92.71 90.17))
+  (wire (pts (xy 67.31 90.17) (xy 72.39 90.17))
     (stroke (width 0) (type default))
   )
   (wire (pts (xy 163.83 101.6) (xy 163.83 97.79))
+    (stroke (width 0) (type default))
+  )
+  (wire (pts (xy 76.2 85.09) (xy 76.2 71.12))
     (stroke (width 0) (type default))
   )
@@
   (symbol (lib_id "Device:R_Small_US") (at 170.18 97.79 90) (unit 1)
     (in_bom yes) (on_board yes) (dnp no) (fields_autoplaced)
-    (property "Reference" "R26" (at 170.18 91.44 90)
+    (property "Reference" "R27" (at 170.18 91.44 90)
       (effects (font (size 1.27 1.27)))
     )
@@
       (project "BTL_ESD"
         (path "/ce4779b4-6d78-42e3-84df-0a4e77629b0f/5a62b24e-983b-422f-a5b4-3f2d2f2b7ed3"
-          (reference "R26") (unit 1)
+          (reference "R27") (unit 1)
         )
       )
@@
   (symbol (lib_id "Device:R_US") (at 226.06 102.87 90) (unit 1)
     (in_bom yes) (on_board yes) (dnp no) (fields_autoplaced)
-    (property "Reference" "R29" (at 226.06 96.52 90)
+    (property "Reference" "R30" (at 226.06 96.52 90)
       (effects (font (size 1.27 1.27)))
     )
@@
       (project "BTL_ESD"
         (path "/ce4779b4-6d78-42e3-84df-0a4e77629b0f/5a62b24e-983b-422f-a5b4-3f2d2f2b7ed3"
-          (reference "R29") (unit 1)
+          (reference "R30") (unit 1)
         )
       )
@@
   (symbol (lib_id "Device:R_US") (at 226.06 77.47 90) (unit 1)
     (in_bom yes) (on_board yes) (dnp no) (fields_autoplaced)
-    (property "Reference" "R28" (at 226.06 71.12 90)
+    (property "Reference" "R29" (at 226.06 71.12 90)
       (effects (font (size 1.27 1.27)))
     )
@@
       (project "BTL_ESD"
         (path "/ce4779b4-6d78-42e3-84df-0a4e77629b0f/5a62b24e-983b-422f-a5b4-3f2d2f2b7ed3"
-          (reference "R28") (unit 1)
+          (reference "R29") (unit 1)
         )
       )
@@
   (symbol (lib_id "Connector:USB_B_Micro") (at 59.69 90.17 0) (unit 1)
     (in_bom yes) (on_board yes) (dnp no) (fields_autoplaced)
-    (property "Reference" "J5" (at 59.69 77.47 0)
+    (property "Reference" "J6" (at 59.69 77.47 0)
       (effects (font (size 1.27 1.27)))
     )
@@
       (project "BTL_ESD"
         (path "/ce4779b4-6d78-42e3-84df-0a4e77629b0f/5a62b24e-983b-422f-a5b4-3f2d2f2b7ed3"
-          (reference "J5") (unit 1)
+          (reference "J6") (unit 1)
         )
       )
@@
   (symbol (lib_id "Device:R_Small_US") (at 170.18 107.95 90) (unit 1)
     (in_bom yes) (on_board yes) (dnp no) (fields_autoplaced)
-    (property "Reference" "R27" (at 170.18 101.6 90)
+    (property "Reference" "R28" (at 170.18 101.6 90)
       (effects (font (size 1.27 1.27)))
     )
@@
       (project "BTL_ESD"
         (path "/ce4779b4-6d78-42e3-84df-0a4e77629b0f/5a62b24e-983b-422f-a5b4-3f2d2f2b7ed3"
-          (reference "R27") (unit 1)
-        )
-      )
+          (reference "R28") (unit 1)
+        )
+      )

Commit message: code:ESP32: update uart driver, main.c && hardware file pcb
Parts:
- J6: URL (none) -> https://www.thegioiic.com/cong-usb-micro-b-2-0-dau-cai-5-ch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
- renumbered R27 to R30, R28 to R31, R29 to R32, R30 to R33
Changed lines of the file:
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@@
   (symbol (lib_id "power:GND") (at 82.55 115.57 0) (unit 1)
     (in_bom yes) (on_board yes) (dnp no) (fields_autoplaced)
-    (property "Reference" "#PWR075" (at 82.55 121.92 0)
+    (property "Reference" "#PWR076" (at 82.55 121.92 0)
       (effects (font (size 1.27 1.27)) hide)
     )
@@
       (project "BTL_ESD"
         (path "/ce4779b4-6d78-42e3-84df-0a4e77629b0f/5a62b24e-983b-422f-a5b4-3f2d2f2b7ed3"
-          (reference "#PWR075") (unit 1)
+          (reference "#PWR076") (unit 1)
         )
       )
@@
   (symbol (lib_id "power:GND") (at 154.94 73.66 0) (unit 1)
     (in_bom yes) (on_board yes) (dnp no) (fields_autoplaced)
-    (property "Reference" "#PWR078" (at 154.94 80.01 0)
+    (property "Reference" "#PWR079" (at 154.94 80.01 0)
       (effects (font (size 1.27 1.27)) hide)
     )
@@
       (project "BTL_ESD"
         (path "/ce4779b4-6d78-42e3-84df-0a4e77629b0f/5a62b24e-983b-422f-a5b4-3f2d2f2b7ed3"
-          (reference "#PWR078") (unit 1)
+          (reference "#PWR079") (unit 1)
         )
       )
@@
   (symbol (lib_id "Device:R_Small_US") (at 170.18 97.79 90) (unit 1)
     (in_bom yes) (on_board yes) (dnp no) (fields_autoplaced)
-    (property "Reference" "R27" (at 170.18 91.44 90)
+    (property "Reference" "R30" (at 170.18 91.44 90)
       (effects (font (size 1.27 1.27)))
     )
@@
       (project "BTL_ESD"
         (path "/ce4779b4-6d78-42e3-84df-0a4e77629b0f/5a62b24e-983b-422f-a5b4-3f2d2f2b7ed3"
-          (reference "R27") (unit 1)
+          (reference "R30") (unit 1)
         )
       )
@@
   (symbol (lib_id "Device:R_US") (at 226.06 102.87 90) (unit 1)
     (in_bom yes) (on_board yes) (dnp no) (fields_autoplaced)
-    (property "Reference" "R30" (at 226.06 96.52 90)
+    (property "Reference" "R33" (at 226.06 96.52 90)
       (effects (font (size 1.27 1.27)))
     )
@@
       (project "BTL_ESD"
         (path "/ce4779b4-6d78-42e3-84df-0a4e77629b0f/5a62b24e-983b-422f-a5b4-3f2d2f2b7ed3"
-          (reference "R30") (unit 1)
+          (reference "R33") (unit 1)
         )
       )
@@
   (symbol (lib_id "power:GND") (at 57.15 102.87 0) (unit 1)
     (in_bom yes) (on_board yes) (dnp no) (fields_autoplaced)
-    (property "Reference" "#PWR074" (at 57.15 109.22 0)
+    (property "Reference" "#PWR075" (at 57.15 109.22 0)
       (effects (font (size 1.27 1.27)) hide)
     )
@@
       (project "BTL_ESD"
         (path "/ce4779b4-6d78-42e3-84df-0a4e77629b0f/5a62b24e-983b-422f-a5b4-3f2d2f2b7ed3"
-          (reference "#PWR074") (unit 1)
+          (reference "#PWR075") (unit 1)
         )
       )
@@
   (symbol (lib_id "power:GND") (at 147.32 113.03 0) (unit 1)
     (in_bom yes) (on_board yes) (dnp no) (fields_autoplaced)
-    (property "Reference" "#PWR077" (at 147.32 119.38 0)
+    (property "Reference" "#PWR078" (at 147.32 119.38 0)
       (effects (font (size 1.27 1.27)) hide)
     )
@@
       (project "BTL_ESD"
         (path "/ce4779b4-6d78-42e3-84df-0a4e77629b0f/5a62b24e-983b-422f-a5b4-3f2d2f2b7ed3"
-          (reference "#PWR077") (unit 1)
+          (reference "#PWR078") (unit 1)
         )
       )
@@
   (symbol (lib_id "Device:R_US") (at 226.06 77.47 90) (unit 1)
     (in_bom yes) (on_board yes) (dnp no) (fields_autoplaced)
-    (property "Reference" "R29" (at 226.06 71.12 90)
+    (property "Reference" "R32" (at 226.06 71.12 90)
       (effects (font (size 1.27 1.27)))
     )
@@
       (project "BTL_ESD"
         (path "/ce4779b4-6d78-42e3-84df-0a4e77629b0f/5a62b24e-983b-422f-a5b4-3f2d2f2b7ed3"
-          (reference "R29") (unit 1)
+          (reference "R32") (unit 1)
         )
       )
@@
     )
     (property "Datasheet" "~" (at 63.5 91.44 0)
+      (effects (font (size 1.27 1.27)) hide)
+    )
+    (property "URL" "https://www.thegioiic.com/cong-usb-micro-b-2-0-dau-cai-5-chan-smd-v2" (at 59.69 90.17 0)
       (effects (font (size 1.27 1.27)) hide)
     )
@@
   (symbol (lib_id "power:GND") (at 88.9 82.55 0) (unit 1)
     (in_bom yes) (on_board yes) (dnp no) (fields_autoplaced)
-    (property "Reference" "#PWR076" (at 88.9 88.9 0)
+    (property "Reference" "#PWR077" (at 88.9 88.9 0)
       (effects (font (size 1.27 1.27)) hide)
     )
@@
       (project "BTL_ESD"
         (path "/ce4779b4-6d78-42e3-84df-0a4e77629b0f/5a62b24e-983b-422f-a5b4-3f2d2f2b7ed3"
-          (reference "#PWR076") (unit 1)
+          (reference "#PWR077") (unit 1)
         )
       )
@@
   (symbol (lib_id "power:+5V") (at 187.96 62.23 0) (unit 1)
     (in_bom yes) (on_board yes) (dnp no) (fields_autoplaced)
-    (property "Reference" "#PWR079" (at 187.96 66.04 0)
+    (property "Reference" "#PWR080" (at 187.96 66.04 0)
       (effects (font (size 1.27 1.27)) hide)
     )
@@
       (project "BTL_ESD"
         (path "/ce4779b4-6d78-42e3-84df-0a4e77629b0f/5a62b24e-983b-422f-a5b4-3f2d2f2b7ed3"
-          (reference "#PWR079") (unit 1)
+          (reference "#PWR080") (unit 1)
         )
       )
@@
   (symbol (lib_id "power:GND") (at 187.96 77.47 0) (unit 1)
     (in_bom yes) (on_board yes) (dnp no) (fields_autoplaced)
-    (property "Reference" "#PWR080" (at 187.96 83.82 0)
+    (property "Reference" "#PWR081" (at 187.96 83.82 0)
       (effects (font (size 1.27 1.27)) hide)
     )
@@
       (project "BTL_ESD"
         (path "/ce4779b4-6d78-42e3-84df-0a4e77629b0f/5a62b24e-983b-422f-a5b4-3f2d2f2b7ed3"
-          (reference "#PWR080") (unit 1)
+          (reference "#PWR081") (unit 1)
         )
       )
@@
   (symbol (lib_id "Device:R_Small_US") (at 170.18 107.95 90) (unit 1)
     (in_bom yes) (on_board yes) (dnp no) (fields_autoplaced)
-    (property "Reference" "R28" (at 170.18 101.6 90)
+    (property "Reference" "R31" (at 170.18 101.6 90)
       (effects (font (size 1.27 1.27)))
     )
@@
       (project "BTL_ESD"
         (path "/ce4779b4-6d78-42e3-84df-0a4e77629b0f/5a62b24e-983b-422f-a5b4-3f2d2f2b7ed3"
-          (reference "R28") (unit 1)
-        )
-      )
+          (reference "R31") (unit 1)
+        )
+      )
