File: Hardware/BTL_ESD/USB_TTL.kicad_sch (KiCad schematic)
At the start: 14 parts, among them J6 USB_B_Micro, Q2 MMBT2222A, Q3 MMBT2222A, U8 CH340C

Commit message: update hardware
Other:
- note added: "AUTO SWITCH MODE"
- note added: "TTL"
- note added: "USB"
- moved on the sheet: C55, C56, C57, Q2, Q3, R30, R31, R32, R33, U8
