File: Hardware/BTL_ESD/esp32.kicad_sch (KiCad schematic)
At the start: 1 part, among them U8 ESP32-WROOM-32E__4MB_HIGH_TEM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

Commit message: hardware: ver 1 schematic
Parts:
- added C38, C40, C41: 100nF/16V, Capacitor_SMD:C_0603_1608Metric_Pad1.08x0.95mm_HandSolder, symbol Device:C_Small
- added C39: 22uF/6.3V, Capacitor_SMD:C_0603_1608Metric_Pad1.08x0.95mm_HandSolder, symbol Device:C_Small
- added D8: Green, LED_SMD:LED_0805_2012Metric_Pad1.15x1.40mm_HandSolder, symbol Device:LED
- added R15, R16, R17: 10k/1%, Resistor_SMD:R_0603_1608Metric_Pad0.98x0.95mm_HandSolder, symbol Device:R_Small_US
- added SW3: ENABLE, Button_Switch_SMD:SW_SPST_B3U-1000P, symbol Switch:SW_Push
- added SW4: FLASH, Button_Switch_SMD:SW_SPST_B3U-1000P, symbol Switch:SW_Push
- renumbered U8 to U5
Connections:
- net GND: now reaches U5.1 (GND), U5.15 (GND), U5.38 (GND), U5.39_1 (GND), U5.39_2 (GND), U5.39_3 (GND), U5.39_4 (GND), U5.39_5 (GND), U5.39_6 (GND), U5.39_7 (GND), U5.39_8 (GND), U5.39_9 (GND)
- net GND: now also C38.2, C39.2, C40.1, C41.1, R15.2, SW3.2, SW4.2
- net +3V3: now reaches U5.2 (3V3)
- net +3V3: now also C38.1, C39.1, R16.1, R17.1
- net LED_STATUS: now reaches U5.23 (IO15)
- net LED_STATUS: now also D8.2 (A)
- net Flash: now reaches U5.25 (IO0)
- net Flash: now also C41.2, R17.2, SW4.1
- net RXD: now reaches U5.27 (IO16)
- net TXD: now reaches U5.28 (IO17)
- net EN: now reaches U5.3 (EN)
- net EN: now also C40.2, R16.2, SW3.1
- net U0_N: now reaches U5.34 (RXD0)
- net U0_P: now reaches U5.35 (TXD0)
- new net: D8.1 (K), R15.1
- no-connect marks 0 -> 22
Other:
- title: (none) -> ESP32

Commit message: update
Parts:
- renumbered D8 to D9
Changed lines of the file:
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@@
   (symbol (lib_id "power:GND") (at 237.49 123.19 0) (unit 1)
     (in_bom yes) (on_board yes) (dnp no) (fields_autoplaced)
-    (property "Reference" "#PWR049" (at 237.49 129.54 0)
+    (property "Reference" "#PWR052" (at 237.49 129.54 0)
       (effects (font (size 1.27 1.27)) hide)
     )
@@
       (project "BTL_ESD"
         (path "/ce4779b4-6d78-42e3-84df-0a4e77629b0f/44099a2a-bdde-4bbb-bae9-9fc724f8d252"
+          (reference "#PWR052") (unit 1)
+        )
+      )
+    )
+  )
+  (symbol (lib_id "Device:C_Small") (at 190.5 55.88 0) (unit 1)
+    (in_bom yes) (on_board yes) (dnp no) (fields_autoplaced)
+    (property "Reference" "C39" (at 193.04 54.6163 0)
+      (effects (font (size 1.27 1.27)) (justify left))
+    )
+    (property "Value" "22uF/6.3V" (at 193.04 57.1563 0)
+      (effects (font (size 1.27 1.27)) (justify left))
+    )
+    (property "Footprint" "Capacitor_SMD:C_0603_1608Metric_Pad1.08x0.95mm_HandSolder" (at 190.5 55.88 0)
+      (effects (font (size 1.27 1.27)) hide)
+    )
+    (property "Datasheet" "~" (at 190.5 55.88 0)
+      (effects (font (size 1.27 1.27)) hide)
+    )
+    (property "URL" "https://www.thegioiic.com/tu-gom-0603-22uf-6-3v" (at 190.5 55.88 0)
+      (effects (font (size 1.27 1.27)) hide)
+    )
+    (pin "2")
+    (pin "1")
+    (instances
+      (project "BTL_ESD"
+        (path "/ce4779b4-6d78-42e3-84df-0a4e77629b0f/44099a2a-bdde-4bbb-bae9-9fc724f8d252"
+          (reference "C39") (unit 1)
+        )
+      )
+    )
+  )
+  (symbol (lib_id "Device:R_Small_US") (at 237.49 100.33 0) (unit 1)
+    (in_bom yes) (on_board yes) (dnp no) (fields_autoplaced)
+    (property "Reference" "R17" (at 240.03 99.06 0)
+      (effects (font (size 1.27 1.27)) (justify left))
+    )
+    (property "Value" "10k/1%" (at 240.03 101.6 0)
+      (effects (font (size 1.27 1.27)) (justify left))
+    )
+    (property "Footprint" "Resistor_SMD:R_0603_1608Metric_Pad0.98x0.95mm_HandSolder" (at 237.49 100.33 0)
+      (effects (font (size 1.27 1.27)) hide)
+    )
+    (property "Datasheet" "~" (at 237.49 100.33 0)
+      (effects (font (size 1.27 1.27)) hide)
+    )
+    (property "URL" "https://www.thegioiic.com/dien-tro-10-kohm-0603-1-" (at 237.49 100.33 0)
+      (effects (font (size 1.27 1.27)) hide)
+    )
+    (pin "1")
+    (pin "2")
+    (instances
+      (project "BTL_ESD"
+        (path "/ce4779b4-6d78-42e3-84df-0a4e77629b0f/44099a2a-bdde-4bbb-bae9-9fc724f8d252"
+          (reference "R17") (unit 1)
+        )
+      )
+    )
+  )
+  (symbol (lib_id "power:+3V3") (at 237.49 49.53 0) (unit 1)
+    (in_bom yes) (on_board yes) (dnp no) (fields_autoplaced)
+    (property "Reference" "#PWR049" (at 237.49 53.34 0)
+      (effects (font (size 1.27 1.27)) hide)
+    )
+    (property "Value" "+3V3" (at 237.49 44.45 0)
+      (effects (font (size 1.27 1.27)))
+    )
+    (property "Footprint" "" (at 237.49 49.53 0)
+      (effects (font (size 1.27 1.27)) hide)
+    )
+    (property "Datasheet" "" (at 237.49 49.53 0)
+      (effects (font (size 1.27 1.27)) hide)
+    )
+    (pin "1")
+    (instances
+      (project "BTL_ESD"
+        (path "/ce4779b4-6d78-42e3-84df-0a4e77629b0f/44099a2a-bdde-4bbb-bae9-9fc724f8d252"
           (reference "#PWR049") (unit 1)
         )
@@
     )
   )
-  (symbol (lib_id "Device:C_Small") (at 190.5 55.88 0) (unit 1)
-    (in_bom yes) (on_board yes) (dnp no) (fields_autoplaced)
-    (property "Reference" "C39" (at 193.04 54.6163 0)
-      (effects (font (size 1.27 1.27)) (justify left))
-    )
-    (property "Value" "22uF/6.3V" (at 193.04 57.1563 0)
-      (effects (font (size 1.27 1.27)) (justify left))
-    )
-    (property "Footprint" "Capacitor_SMD:C_0603_1608Metric_Pad1.08x0.95mm_HandSolder" (at 190.5 55.88 0)
-      (effects (font (size 1.27 1.27)) hide)
-    )
-    (property "Datasheet" "~" (at 190.5 55.88 0)
-      (effects (font (size 1.27 1.27)) hide)
-    )
-    (property "URL" "https://www.thegioiic.com/tu-gom-0603-22uf-6-3v" (at 190.5 55.88 0)
-      (effects (font (size 1.27 1.27)) hide)
-    )
-    (pin "2")
-    (pin "1")
-    (instances
-      (project "BTL_ESD"
-        (path "/ce4779b4-6d78-42e3-84df-0a4e77629b0f/44099a2a-bdde-4bbb-bae9-9fc724f8d252"
-          (reference "C39") (unit 1)
-        )
-      )
-    )
-  )
-  (symbol (lib_id "Device:R_Small_US") (at 237.49 100.33 0) (unit 1)
-    (in_bom yes) (on_board yes) (dnp no) (fields_autoplaced)
-    (property "Reference" "R17" (at 240.03 99.06 0)
-      (effects (font (size 1.27 1.27)) (justify left))
-    )
-    (property "Value" "10k/1%" (at 240.03 101.6 0)
-      (effects (font (size 1.27 1.27)) (justify left))
-    )
-    (property "Footprint" "Resistor_SMD:R_0603_1608Metric_Pad0.98x0.95mm_HandSolder" (at 237.49 100.33 0)
-      (effects (font (size 1.27 1.27)) hide)
-    )
-    (property "Datasheet" "~" (at 237.49 100.33 0)
-      (effects (font (size 1.27 1.27)) hide)
-    )
-    (property "URL" "https://www.thegioiic.com/dien-tro-10-kohm-0603-1-" (at 237.49 100.33 0)
-      (effects (font (size 1.27 1.27)) hide)
-    )
-    (pin "1")
-    (pin "2")
-    (instances
-      (project "BTL_ESD"
-        (path "/ce4779b4-6d78-42e3-84df-0a4e77629b0f/44099a2a-bdde-4bbb-bae9-9fc724f8d252"
-          (reference "R17") (unit 1)
-        )
-      )
-    )
-  )
-  (symbol (lib_id "power:+3V3") (at 237.49 49.53 0) (unit 1)
-    (in_bom yes) (on_board yes) (dnp no) (fields_autoplaced)
-    (property "Reference" "#PWR046" (at 237.49 53.34 0)
-      (effects (font (size 1.27 1.27)) hide)
-    )
-    (property "Value" "+3V3" (at 237.49 44.45 0)
-      (effects (font (size 1.27 1.27)))
-    )
-    (property "Footprint" "" (at 237.49 49.53 0)
-      (effects (font (size 1.27 1.27)) hide)
-    )
-    (property "Datasheet" "" (at 237.49 49.53 0)
-      (effects (font (size 1.27 1.27)) hide)
-    )
-    (pin "1")
-    (instances
-      (project "BTL_ESD"
-        (path "/ce4779b4-6d78-42e3-84df-0a4e77629b0f/44099a2a-bdde-4bbb-bae9-9fc724f8d252"
-          (reference "#PWR046") (unit 1)
-        )
-      )
-    )
-  )
   (symbol (lib_id "Device:R_Small_US") (at 154.94 140.97 90) (unit 1)
     (in_bom yes) (on_board yes) (dnp no) (fields_autoplaced)
@@
   (symbol (lib_id "power:GND") (at 182.88 62.23 0) (unit 1)
     (in_bom yes) (on_board yes) (dnp no) (fields_autoplaced)
-    (property "Reference" "#PWR045" (at 182.88 68.58 0)
+    (property "Reference" "#PWR048" (at 182.88 68.58 0)
       (effects (font (size 1.27 1.27)) hide)
     )
@@
       (project "BTL_ESD"
         (path "/ce4779b4-6d78-42e3-84df-0a4e77629b0f/44099a2a-bdde-4bbb-bae9-9fc724f8d252"
-          (reference "#PWR045") (unit 1)
+          (reference "#PWR048") (unit 1)
         )
       )
@@
   (symbol (lib_id "power:GND") (at 170.18 124.46 0) (unit 1)
     (in_bom yes) (on_board yes) (dnp no) (fields_autoplaced)
-    (property "Reference" "#PWR043" (at 170.18 130.81 0)
+    (property "Reference" "#PWR046" (at 170.18 130.81 0)
       (effects (font (size 1.27 1.27)) hide)
     )
@@
       (project "BTL_ESD"
         (path "/ce4779b4-6d78-42e3-84df-0a4e77629b0f/44099a2a-bdde-4bbb-bae9-9fc724f8d252"
-          (reference "#PWR043") (unit 1)
+          (reference "#PWR046") (unit 1)
         )
       )
@@
   (symbol (lib_id "Device:LED") (at 143.51 140.97 180) (unit 1)
     (in_bom yes) (on_board yes) (dnp no)
-    (property "Reference" "D8" (at 143.51 135.89 0)
+    (property "Reference" "D9" (at 143.51 135.89 0)
       (effects (font (size 1.27 1.27)))
     )
@@
       (project "BTL_ESD"
         (path "/ce4779b4-6d78-42e3-84df-0a4e77629b0f/44099a2a-bdde-4bbb-bae9-9fc724f8d252"
-          (reference "D8") (unit 1)
+          (reference "D9") (unit 1)
         )
       )
@@
   (symbol (lib_id "power:+3V3") (at 237.49 93.98 0) (unit 1)
     (in_bom yes) (on_board yes) (dnp no) (fields_autoplaced)
-    (property "Reference" "#PWR048" (at 237.49 97.79 0)
+    (property "Reference" "#PWR051" (at 237.49 97.79 0)
       (effects (font (size 1.27 1.27)) hide)
     )
@@
       (project "BTL_ESD"
         (path "/ce4779b4-6d78-42e3-84df-0a4e77629b0f/44099a2a-bdde-4bbb-bae9-9fc724f8d252"
-          (reference "#PWR048") (unit 1)
+          (reference "#PWR051") (unit 1)
         )
       )
@@
   (symbol (lib_id "power:+3V3") (at 182.88 49.53 0) (unit 1)
     (in_bom yes) (on_board yes) (dnp no) (fields_autoplaced)
-    (property "Reference" "#PWR044" (at 182.88 53.34 0)
+    (property "Reference" "#PWR047" (at 182.88 53.34 0)
       (effects (font (size 1.27 1.27)) hide)
     )
@@
       (project "BTL_ESD"
         (path "/ce4779b4-6d78-42e3-84df-0a4e77629b0f/44099a2a-bdde-4bbb-bae9-9fc724f8d252"
-          (reference "#PWR044") (unit 1)
+          (reference "#PWR047") (unit 1)
         )
       )
@@
   (symbol (lib_id "power:GND") (at 161.29 143.51 0) (unit 1)
     (in_bom yes) (on_board yes) (dnp no) (fields_autoplaced)
-    (property "Reference" "#PWR042" (at 161.29 149.86 0)
+    (property "Reference" "#PWR045" (at 161.29 149.86 0)
       (effects (font (size 1.27 1.27)) hide)
     )
@@
       (project "BTL_ESD"
         (path "/ce4779b4-6d78-42e3-84df-0a4e77629b0f/44099a2a-bdde-4bbb-bae9-9fc724f8d252"
-          (reference "#PWR042") (unit 1)
+          (reference "#PWR045") (unit 1)
         )
       )
@@
   (symbol (lib_id "power:GND") (at 237.49 78.74 0) (unit 1)
     (in_bom yes) (on_board yes) (dnp no) (fields_autoplaced)
-    (property "Reference" "#PWR047" (at 237.49 85.09 0)
+    (property "Reference" "#PWR050" (at 237.49 85.09 0)
       (effects (font (size 1.27 1.27)) hide)
     )
@@
       (project "BTL_ESD"
         (path "/ce4779b4-6d78-42e3-84df-0a4e77629b0f/44099a2a-bdde-4bbb-bae9-9fc724f8d252"
-          (reference "#PWR047") (unit 1)
-        )
-      )
+          (reference "#PWR050") (unit 1)
+        )
+      )

Commit message: fea:STM32: upload structure fodler
Parts:
- renumbered R15 to R16, R16 to R17, R17 to R18
Connections:
- net GPIO_1: now reaches U5.14 (IO12)
- net GPIO_2: now reaches U5.16 (IO13)
- net Flash renamed FLASH
- net RXD renamed RXD_2
- net TXD renamed TXD_2
- no-connect marks 22 -> 20
Changed lines of the file:
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@@
   (no_connect (at 165.1 101.6))
   (no_connect (at 165.1 71.12))
-  (no_connect (at 165.1 81.28))
   (no_connect (at 165.1 106.68))
   (no_connect (at 165.1 76.2))
@@
   (no_connect (at 124.46 106.68))
   (no_connect (at 165.1 96.52))
-  (no_connect (at 165.1 78.74))
   (no_connect (at 165.1 99.06))
   (wire (pts (xy 182.88 86.36) (xy 165.1 86.36))
@@
     (stroke (width 0) (type default))
   )
+  (wire (pts (xy 171.45 78.74) (xy 165.1 78.74))
+    (stroke (width 0) (type default))
+  )
   (wire (pts (xy 182.88 52.07) (xy 190.5 52.07))
     (stroke (width 0) (type default))
@@
     (stroke (width 0) (type default))
   )
+  (wire (pts (xy 165.1 81.28) (xy 171.45 81.28))
+    (stroke (width 0) (type default))
+  )
   (wire (pts (xy 237.49 120.65) (xy 237.49 123.19))
     (stroke (width 0) (type default))
@@
     (stroke (width 0) (type default))
   )
-  (wire (pts (xy 168.91 68.58) (xy 165.1 68.58))
+  (wire (pts (xy 170.18 68.58) (xy 165.1 68.58))
     (stroke (width 0) (type default))
   )
@@
     )
   )
-  (global_label "Flash" (shape bidirectional) (at 168.91 68.58 0) (fields_autoplaced)
-    (effects (font (size 1.27 1.27)) (justify left))
-    (property "Intersheetrefs" "${INTERSHEET_REFS}" (at 178.0864 68.58 0)
-      (effects (font (size 1.27 1.27)) (justify left) hide)
-    )
-  )
   (global_label "U0_P" (shape output) (at 119.38 96.52 180) (fields_autoplaced)
     (effects (font (size 1.27 1.27)) (justify right))
@@
     )
   )
-  (global_label "RXD" (shape input) (at 170.18 88.9 0) (fields_autoplaced)
+  (global_label "GPIO_1" (shape bidirectional) (at 171.45 78.74 0) (fields_autoplaced)
     (effects (font (size 1.27 1.27)) (justify left))
-    (property "Intersheetrefs" "${INTERSHEET_REFS}" (at 176.9147 88.9 0)
+    (property "Intersheetrefs" "${INTERSHEET_REFS}" (at 182.1989 78.74 0)
+      (effects (font (size 1.27 1.27)) (justify left) hide)
+    )
+  )
+  (global_label "RXD_2" (shape input) (at 170.18 88.9 0) (fields_autoplaced)
+    (effects (font (size 1.27 1.27)) (justify left))
+    (property "Intersheetrefs" "${INTERSHEET_REFS}" (at 179.0918 88.9 0)
+      (effects (font (size 1.27 1.27)) (justify left) hide)
+    )
+  )
+  (global_label "GPIO_2" (shape bidirectional) (at 171.45 81.28 0) (fields_autoplaced)
+    (effects (font (size 1.27 1.27)) (justify left))
+    (property "Intersheetrefs" "${INTERSHEET_REFS}" (at 182.1989 81.28 0)
       (effects (font (size 1.27 1.27)) (justify left) hide)
     )
@@
     )
   )
-  (global_label "Flash" (shape bidirectional) (at 233.68 105.41 180) (fields_autoplaced)
-    (effects (font (size 1.27 1.27)) (justify right))
-    (property "Intersheetrefs" "${INTERSHEET_REFS}" (at 224.5036 105.41 0)
-      (effects (font (size 1.27 1.27)) (justify right) hide)
-    )
-  )
-  (global_label "TXD" (shape output) (at 171.45 91.44 0) (fields_autoplaced)
+  (global_label "FLASH" (shape bidirectional) (at 170.18 68.58 0) (fields_autoplaced)
     (effects (font (size 1.27 1.27)) (justify left))
-    (property "Intersheetrefs" "${INTERSHEET_REFS}" (at 177.8823 91.44 0)
+    (property "Intersheetrefs" "${INTERSHEET_REFS}" (at 180.0218 68.58 0)
+      (effects (font (size 1.27 1.27)) (justify left) hide)
+    )
+  )
+  (global_label "TXD_2" (shape output) (at 171.45 91.44 0) (fields_autoplaced)
+    (effects (font (size 1.27 1.27)) (justify left))
+    (property "Intersheetrefs" "${INTERSHEET_REFS}" (at 180.0594 91.44 0)
       (effects (font (size 1.27 1.27)) (justify left) hide)
     )
@@
     )
   )
+  (global_label "FLASH" (shape bidirectional) (at 233.68 105.41 180) (fields_autoplaced)
+    (effects (font (size 1.27 1.27)) (justify right))
+    (property "Intersheetrefs" "${INTERSHEET_REFS}" (at 223.8382 105.41 0)
+      (effects (font (size 1.27 1.27)) (justify right) hide)
+    )
+  )
   (symbol (lib_id "power:GND") (at 237.49 123.19 0) (unit 1)
     (in_bom yes) (on_board yes) (dnp no) (fields_autoplaced)
@@
   (symbol (lib_id "Device:R_Small_US") (at 237.49 100.33 0) (unit 1)
     (in_bom yes) (on_board yes) (dnp no) (fields_autoplaced)
-    (property "Reference" "R17" (at 240.03 99.06 0)
+    (property "Reference" "R18" (at 240.03 99.06 0)
       (effects (font (size 1.27 1.27)) (justify left))
     )
@@
       (project "BTL_ESD"
         (path "/ce4779b4-6d78-42e3-84df-0a4e77629b0f/44099a2a-bdde-4bbb-bae9-9fc724f8d252"
-          (reference "R17") (unit 1)
+          (reference "R18") (unit 1)
         )
       )
@@
   (symbol (lib_id "Device:R_Small_US") (at 154.94 140.97 90) (unit 1)
     (in_bom yes) (on_board yes) (dnp no) (fields_autoplaced)
-    (property "Reference" "R15" (at 154.94 134.62 90)
+    (property "Reference" "R16" (at 154.94 134.62 90)
       (effects (font (size 1.27 1.27)))
     )
@@
       (project "BTL_ESD"
         (path "/ce4779b4-6d78-42e3-84df-0a4e77629b0f/44099a2a-bdde-4bbb-bae9-9fc724f8d252"
-          (reference "R15") (unit 1)
+          (reference "R16") (unit 1)
         )
       )
@@
   (symbol (lib_id "Device:R_Small_US") (at 237.49 55.88 0) (unit 1)
     (in_bom yes) (on_board yes) (dnp no) (fields_autoplaced)
-    (property "Reference" "R16" (at 240.03 54.61 0)
+    (property "Reference" "R17" (at 240.03 54.61 0)
       (effects (font (size 1.27 1.27)) (justify left))
     )
@@
       (project "BTL_ESD"
         (path "/ce4779b4-6d78-42e3-84df-0a4e77629b0f/44099a2a-bdde-4bbb-bae9-9fc724f8d252"
-          (reference "R16") (unit 1)
-        )
-      )
+          (reference "R17") (unit 1)
+        )
+      )
