File: Hardware/BTL_ESD/measure.kicad_sch (KiCad schematic)
At the start: 1 part, among them U4 INA128

Commit message: hardware: ver 1 schematic
Parts:
- removed U4: INA128, symbol Amplifier_Instrumentation:INA128
- added C48: 1uF/16V, Capacitor_SMD:C_0603_1608Metric_Pad1.08x0.95mm_HandSolder, symbol Device:C_Small
- added C49, C50: 10uF/16V, Capacitor_SMD:C_0603_1608Metric_Pad1.08x0.95mm_HandSolder, symbol Device:C_Small
- added C51, C52: 100nF/16V, Capacitor_SMD:C_0603_1608Metric_Pad1.08x0.95mm_HandSolder, symbol Device:C_Small
- added R24: GL5528, Resistor_THT:R_Axial_DIN0516_L15.5mm_D5.0mm_P5.08mm_Vertical, symbol Device:R_Variable_US
- added TP5: V_P, TestPoint:TestPoint_Pad_D2.5mm, symbol Connector:TestPoint
- added TP6: V_N, TestPoint:TestPoint_Pad_D2.5mm, symbol Connector:TestPoint
- added U7: INA128UA, INA128UA:SOIC127P599X175-8N, symbol INA128UA:INA128UA
- added VR1, VR2: 50k/0.15W, footprints:EVM-3E, symbol EVM_3E:EVM-3E
Connections:
- new net: U7.1 (RG), VR2.2
- new net: U7.8 (RG), VR2.1
- new net +5V: C49.1, C51.1, U7.7 (V+)
- new net -5V: C50.1, C52.1, U7.4 (V-)
- new net ADC1_0: U7.6 (VO)
- new net CURRENT_SUPPLY: C48.1, R24.1, TP5.1, U7.3 (V+IN), VR1.2
- new net GND: C48.2, C49.2, C50.2, C51.2, C52.2, R24.2, TP6.1, U7.2 (V-IN), U7.5 (REF), VR1.1
- no-connect marks 0 -> 2
Other:
- title: (none) -> MEASURE

Commit message: update
Parts:
- added TP7: RG_1, TestPoint:TestPoint_Pad_D2.5mm, symbol Connector:TestPoint
- added TP8: RG_2, TestPoint:TestPoint_Pad_D2.5mm, symbol Connector:TestPoint
- R24: footprint Resistor_THT:R_Axial_DIN0516_L15.5mm_D5.0mm_P5.08mm_Vertical -> OptoDevice:R_LDR_5.0x4.1mm_P3mm_Vertical
Connections:
- net at U7.1 (RG), VR2.2: now also TP7.1
- net at U7.8 (RG), VR2.1: now also TP8.1
- net GND renamed GNDA
Other:
- moved on the sheet: VR2

Commit message: update
Parts:
- renumbered R24 to R25

Commit message: fea:STM32: upload structure fodler
Parts:
- renumbered R25 to R26
Changed lines of the file:
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@@
   (symbol (lib_id "Device:R_Variable_US") (at 101.6 97.79 0) (unit 1)
     (in_bom yes) (on_board yes) (dnp no) (fields_autoplaced)
-    (property "Reference" "R25" (at 105.41 96.4819 0)
+    (property "Reference" "R26" (at 105.41 96.4819 0)
       (effects (font (size 1.27 1.27)) (justify left))
     )
@@
       (project "BTL_ESD"
         (path "/ce4779b4-6d78-42e3-84df-0a4e77629b0f/c3280f20-486c-46c2-9703-f7181f16559f"
-          (reference "R25") (unit 1)
+          (reference "R26") (unit 1)
         )
       )

Commit message: hardware:update pcb track power
Parts:
- renumbered TP5 to TP6, TP6 to TP7, TP7 to TP8, TP8 to TP9
Changed lines of the file:
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@@
   (symbol (lib_id "Connector:TestPoint") (at 91.44 91.44 0) (unit 1)
     (in_bom yes) (on_board yes) (dnp no) (fields_autoplaced)
-    (property "Reference" "TP5" (at 93.98 86.868 0)
+    (property "Reference" "TP6" (at 93.98 86.868 0)
       (effects (font (size 1.27 1.27)) (justify left))
     )
@@
       (project "BTL_ESD"
         (path "/ce4779b4-6d78-42e3-84df-0a4e77629b0f/c3280f20-486c-46c2-9703-f7181f16559f"
-          (reference "TP5") (unit 1)
+          (reference "TP6") (unit 1)
         )
       )
@@
   (symbol (lib_id "power:+5V") (at 228.6 62.23 0) (unit 1)
     (in_bom yes) (on_board yes) (dnp no) (fields_autoplaced)
-    (property "Reference" "#PWR069" (at 228.6 66.04 0)
+    (property "Reference" "#PWR070" (at 228.6 66.04 0)
       (effects (font (size 1.27 1.27)) hide)
     )
@@
       (project "BTL_ESD"
         (path "/ce4779b4-6d78-42e3-84df-0a4e77629b0f/c3280f20-486c-46c2-9703-f7181f16559f"
+          (reference "#PWR070") (unit 1)
+        )
+      )
+    )
+  )
+  (symbol (lib_id "power:-5V") (at 181.61 97.79 0) (unit 1)
+    (in_bom yes) (on_board yes) (dnp no) (fields_autoplaced)
+    (property "Reference" "#PWR069" (at 181.61 95.25 0)
+      (effects (font (size 1.27 1.27)) hide)
+    )
+    (property "Value" "-5V" (at 181.61 92.71 0)
+      (effects (font (size 1.27 1.27)))
+    )
+    (property "Footprint" "" (at 181.61 97.79 0)
+      (effects (font (size 1.27 1.27)) hide)
+    )
+    (property "Datasheet" "" (at 181.61 97.79 0)
+      (effects (font (size 1.27 1.27)) hide)
+    )
+    (pin "1")
+    (instances
+      (project "BTL_ESD"
+        (path "/ce4779b4-6d78-42e3-84df-0a4e77629b0f/c3280f20-486c-46c2-9703-f7181f16559f"
           (reference "#PWR069") (unit 1)
         )
@@
     )
   )
-  (symbol (lib_id "power:-5V") (at 181.61 97.79 0) (unit 1)
-    (in_bom yes) (on_board yes) (dnp no) (fields_autoplaced)
-    (property "Reference" "#PWR068" (at 181.61 95.25 0)
-      (effects (font (size 1.27 1.27)) hide)
-    )
-    (property "Value" "-5V" (at 181.61 92.71 0)
-      (effects (font (size 1.27 1.27)))
-    )
-    (property "Footprint" "" (at 181.61 97.79 0)
-      (effects (font (size 1.27 1.27)) hide)
-    )
-    (property "Datasheet" "" (at 181.61 97.79 0)
-      (effects (font (size 1.27 1.27)) hide)
-    )
-    (pin "1")
-    (instances
-      (project "BTL_ESD"
-        (path "/ce4779b4-6d78-42e3-84df-0a4e77629b0f/c3280f20-486c-46c2-9703-f7181f16559f"
-          (reference "#PWR068") (unit 1)
-        )
-      )
-    )
-  )
   (symbol (lib_id "Connector:TestPoint") (at 133.35 90.17 0) (unit 1)
     (in_bom yes) (on_board yes) (dnp no) (fields_autoplaced)
-    (property "Reference" "TP8" (at 135.89 85.598 0)
+    (property "Reference" "TP9" (at 135.89 85.598 0)
       (effects (font (size 1.27 1.27)) (justify left))
     )
@@
       (project "BTL_ESD"
         (path "/ce4779b4-6d78-42e3-84df-0a4e77629b0f/c3280f20-486c-46c2-9703-f7181f16559f"
-          (reference "TP8") (unit 1)
+          (reference "TP9") (unit 1)
         )
       )
@@
   (symbol (lib_id "Connector:TestPoint") (at 91.44 102.87 0) (unit 1)
     (in_bom yes) (on_board yes) (dnp no) (fields_autoplaced)
-    (property "Reference" "TP6" (at 93.98 98.298 0)
+    (property "Reference" "TP7" (at 93.98 98.298 0)
       (effects (font (size 1.27 1.27)) (justify left))
     )
@@
       (project "BTL_ESD"
         (path "/ce4779b4-6d78-42e3-84df-0a4e77629b0f/c3280f20-486c-46c2-9703-f7181f16559f"
-          (reference "TP6") (unit 1)
+          (reference "TP7") (unit 1)
         )
       )
@@
   (symbol (lib_id "power:GNDA") (at 142.24 105.41 0) (unit 1)
     (in_bom yes) (on_board yes) (dnp no) (fields_autoplaced)
-    (property "Reference" "#PWR066" (at 142.24 111.76 0)
+    (property "Reference" "#PWR067" (at 142.24 111.76 0)
       (effects (font (size 1.27 1.27)) hide)
     )
@@
       (project "BTL_ESD"
         (path "/ce4779b4-6d78-42e3-84df-0a4e77629b0f/c3280f20-486c-46c2-9703-f7181f16559f"
-          (reference "#PWR066") (unit 1)
+          (reference "#PWR067") (unit 1)
         )
       )
@@
   (symbol (lib_id "power:GNDA") (at 101.6 111.76 0) (unit 1)
     (in_bom yes) (on_board yes) (dnp no) (fields_autoplaced)
-    (property "Reference" "#PWR065" (at 101.6 118.11 0)
+    (property "Reference" "#PWR066" (at 101.6 118.11 0)
       (effects (font (size 1.27 1.27)) hide)
     )
@@
       (project "BTL_ESD"
         (path "/ce4779b4-6d78-42e3-84df-0a4e77629b0f/c3280f20-486c-46c2-9703-f7181f16559f"
-          (reference "#PWR065") (unit 1)
+          (reference "#PWR066") (unit 1)
         )
       )
@@
   (symbol (lib_id "Connector:TestPoint") (at 133.35 78.74 0) (unit 1)
     (in_bom yes) (on_board yes) (dnp no) (fields_autoplaced)
-    (property "Reference" "TP7" (at 135.89 74.168 0)
+    (property "Reference" "TP8" (at 135.89 74.168 0)
       (effects (font (size 1.27 1.27)) (justify left))
     )
@@
       (project "BTL_ESD"
         (path "/ce4779b4-6d78-42e3-84df-0a4e77629b0f/c3280f20-486c-46c2-9703-f7181f16559f"
-          (reference "TP7") (unit 1)
+          (reference "TP8") (unit 1)
         )
       )
@@
   (symbol (lib_id "power:GNDA") (at 228.6 110.49 0) (unit 1)
     (in_bom yes) (on_board yes) (dnp no) (fields_autoplaced)
-    (property "Reference" "#PWR072" (at 228.6 116.84 0)
+    (property "Reference" "#PWR073" (at 228.6 116.84 0)
       (effects (font (size 1.27 1.27)) hide)
     )
@@
       (project "BTL_ESD"
         (path "/ce4779b4-6d78-42e3-84df-0a4e77629b0f/c3280f20-486c-46c2-9703-f7181f16559f"
-          (reference "#PWR072") (unit 1)
+          (reference "#PWR073") (unit 1)
         )
       )
@@
   (symbol (lib_id "power:GNDA") (at 228.6 74.93 0) (unit 1)
     (in_bom yes) (on_board yes) (dnp no) (fields_autoplaced)
-    (property "Reference" "#PWR070" (at 228.6 81.28 0)
+    (property "Reference" "#PWR071" (at 228.6 81.28 0)
       (effects (font (size 1.27 1.27)) hide)
     )
@@
       (project "BTL_ESD"
         (path "/ce4779b4-6d78-42e3-84df-0a4e77629b0f/c3280f20-486c-46c2-9703-f7181f16559f"
-          (reference "#PWR070") (unit 1)
+          (reference "#PWR071") (unit 1)
         )
       )
@@
   (symbol (lib_id "power:-5V") (at 228.6 97.79 0) (unit 1)
     (in_bom yes) (on_board yes) (dnp no) (fields_autoplaced)
-    (property "Reference" "#PWR071" (at 228.6 95.25 0)
+    (property "Reference" "#PWR072" (at 228.6 95.25 0)
       (effects (font (size 1.27 1.27)) hide)
     )
@@
       (project "BTL_ESD"
         (path "/ce4779b4-6d78-42e3-84df-0a4e77629b0f/c3280f20-486c-46c2-9703-f7181f16559f"
-          (reference "#PWR071") (unit 1)
+          (reference "#PWR072") (unit 1)
         )
       )
@@
   (symbol (lib_id "power:+5V") (at 181.61 77.47 0) (unit 1)
     (in_bom yes) (on_board yes) (dnp no) (fields_autoplaced)
-    (property "Reference" "#PWR067" (at 181.61 81.28 0)
+    (property "Reference" "#PWR068" (at 181.61 81.28 0)
       (effects (font (size 1.27 1.27)) hide)
     )
@@
       (project "BTL_ESD"
         (path "/ce4779b4-6d78-42e3-84df-0a4e77629b0f/c3280f20-486c-46c2-9703-f7181f16559f"
-          (reference "#PWR067") (unit 1)
-        )
-      )
+          (reference "#PWR068") (unit 1)
+        )
+      )

Commit message: code:ESP32: update uart driver, main.c && hardware file pcb
Parts:
- renumbered R26 to R29
Changed lines of the file:
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@@
   (symbol (lib_id "power:+5V") (at 228.6 62.23 0) (unit 1)
     (in_bom yes) (on_board yes) (dnp no) (fields_autoplaced)
-    (property "Reference" "#PWR070" (at 228.6 66.04 0)
+    (property "Reference" "#PWR071" (at 228.6 66.04 0)
       (effects (font (size 1.27 1.27)) hide)
     )
@@
       (project "BTL_ESD"
         (path "/ce4779b4-6d78-42e3-84df-0a4e77629b0f/c3280f20-486c-46c2-9703-f7181f16559f"
+          (reference "#PWR071") (unit 1)
+        )
+      )
+    )
+  )
+  (symbol (lib_id "power:-5V") (at 181.61 97.79 0) (unit 1)
+    (in_bom yes) (on_board yes) (dnp no) (fields_autoplaced)
+    (property "Reference" "#PWR070" (at 181.61 95.25 0)
+      (effects (font (size 1.27 1.27)) hide)
+    )
+    (property "Value" "-5V" (at 181.61 92.71 0)
+      (effects (font (size 1.27 1.27)))
+    )
+    (property "Footprint" "" (at 181.61 97.79 0)
+      (effects (font (size 1.27 1.27)) hide)
+    )
+    (property "Datasheet" "" (at 181.61 97.79 0)
+      (effects (font (size 1.27 1.27)) hide)
+    )
+    (pin "1")
+    (instances
+      (project "BTL_ESD"
+        (path "/ce4779b4-6d78-42e3-84df-0a4e77629b0f/c3280f20-486c-46c2-9703-f7181f16559f"
           (reference "#PWR070") (unit 1)
         )
@@
     )
   )
-  (symbol (lib_id "power:-5V") (at 181.61 97.79 0) (unit 1)
-    (in_bom yes) (on_board yes) (dnp no) (fields_autoplaced)
-    (property "Reference" "#PWR069" (at 181.61 95.25 0)
-      (effects (font (size 1.27 1.27)) hide)
-    )
-    (property "Value" "-5V" (at 181.61 92.71 0)
-      (effects (font (size 1.27 1.27)))
-    )
-    (property "Footprint" "" (at 181.61 97.79 0)
-      (effects (font (size 1.27 1.27)) hide)
-    )
-    (property "Datasheet" "" (at 181.61 97.79 0)
-      (effects (font (size 1.27 1.27)) hide)
-    )
-    (pin "1")
-    (instances
-      (project "BTL_ESD"
-        (path "/ce4779b4-6d78-42e3-84df-0a4e77629b0f/c3280f20-486c-46c2-9703-f7181f16559f"
-          (reference "#PWR069") (unit 1)
-        )
-      )
-    )
-  )
   (symbol (lib_id "Connector:TestPoint") (at 133.35 90.17 0) (unit 1)
     (in_bom yes) (on_board yes) (dnp no) (fields_autoplaced)
@@
   (symbol (lib_id "power:GNDA") (at 142.24 105.41 0) (unit 1)
     (in_bom yes) (on_board yes) (dnp no) (fields_autoplaced)
-    (property "Reference" "#PWR067" (at 142.24 111.76 0)
+    (property "Reference" "#PWR068" (at 142.24 111.76 0)
       (effects (font (size 1.27 1.27)) hide)
     )
@@
       (project "BTL_ESD"
         (path "/ce4779b4-6d78-42e3-84df-0a4e77629b0f/c3280f20-486c-46c2-9703-f7181f16559f"
-          (reference "#PWR067") (unit 1)
+          (reference "#PWR068") (unit 1)
         )
       )
@@
   (symbol (lib_id "power:GNDA") (at 101.6 111.76 0) (unit 1)
     (in_bom yes) (on_board yes) (dnp no) (fields_autoplaced)
-    (property "Reference" "#PWR066" (at 101.6 118.11 0)
+    (property "Reference" "#PWR067" (at 101.6 118.11 0)
       (effects (font (size 1.27 1.27)) hide)
     )
@@
       (project "BTL_ESD"
         (path "/ce4779b4-6d78-42e3-84df-0a4e77629b0f/c3280f20-486c-46c2-9703-f7181f16559f"
-          (reference "#PWR066") (unit 1)
+          (reference "#PWR067") (unit 1)
         )
       )
@@
   (symbol (lib_id "power:GNDA") (at 228.6 110.49 0) (unit 1)
     (in_bom yes) (on_board yes) (dnp no) (fields_autoplaced)
-    (property "Reference" "#PWR073" (at 228.6 116.84 0)
+    (property "Reference" "#PWR074" (at 228.6 116.84 0)
       (effects (font (size 1.27 1.27)) hide)
     )
@@
       (project "BTL_ESD"
         (path "/ce4779b4-6d78-42e3-84df-0a4e77629b0f/c3280f20-486c-46c2-9703-f7181f16559f"
-          (reference "#PWR073") (unit 1)
+          (reference "#PWR074") (unit 1)
         )
       )
@@
   (symbol (lib_id "power:GNDA") (at 228.6 74.93 0) (unit 1)
     (in_bom yes) (on_board yes) (dnp no) (fields_autoplaced)
-    (property "Reference" "#PWR071" (at 228.6 81.28 0)
+    (property "Reference" "#PWR072" (at 228.6 81.28 0)
       (effects (font (size 1.27 1.27)) hide)
     )
@@
       (project "BTL_ESD"
         (path "/ce4779b4-6d78-42e3-84df-0a4e77629b0f/c3280f20-486c-46c2-9703-f7181f16559f"
-          (reference "#PWR071") (unit 1)
+          (reference "#PWR072") (unit 1)
         )
       )
@@
   (symbol (lib_id "power:-5V") (at 228.6 97.79 0) (unit 1)
     (in_bom yes) (on_board yes) (dnp no) (fields_autoplaced)
-    (property "Reference" "#PWR072" (at 228.6 95.25 0)
+    (property "Reference" "#PWR073" (at 228.6 95.25 0)
       (effects (font (size 1.27 1.27)) hide)
     )
@@
       (project "BTL_ESD"
         (path "/ce4779b4-6d78-42e3-84df-0a4e77629b0f/c3280f20-486c-46c2-9703-f7181f16559f"
-          (reference "#PWR072") (unit 1)
+          (reference "#PWR073") (unit 1)
         )
       )
@@
   (symbol (lib_id "Device:R_Variable_US") (at 101.6 97.79 0) (unit 1)
     (in_bom yes) (on_board yes) (dnp no) (fields_autoplaced)
-    (property "Reference" "R26" (at 105.41 96.4819 0)
+    (property "Reference" "R29" (at 105.41 96.4819 0)
       (effects (font (size 1.27 1.27)) (justify left))
     )
@@
       (project "BTL_ESD"
         (path "/ce4779b4-6d78-42e3-84df-0a4e77629b0f/c3280f20-486c-46c2-9703-f7181f16559f"
-          (reference "R26") (unit 1)
+          (reference "R29") (unit 1)
         )
       )
@@
   (symbol (lib_id "power:+5V") (at 181.61 77.47 0) (unit 1)
     (in_bom yes) (on_board yes) (dnp no) (fields_autoplaced)
-    (property "Reference" "#PWR068" (at 181.61 81.28 0)
+    (property "Reference" "#PWR069" (at 181.61 81.28 0)
       (effects (font (size 1.27 1.27)) hide)
     )
@@
       (project "BTL_ESD"
         (path "/ce4779b4-6d78-42e3-84df-0a4e77629b0f/c3280f20-486c-46c2-9703-f7181f16559f"
-          (reference "#PWR068") (unit 1)
-        )
-      )
+          (reference "#PWR069") (unit 1)
+        )
+      )
