File: Hardware/BTL_ESD/measure.kicad_sch (KiCad schematic)
At the start: 13 parts, among them U7 INA128UA

Commit message: update hardware
Connections:
- net ADC1_0 renamed ADC2_0
Other:
- note added: "FILTER"
- note added: "MEASURE RESISTOR"
- moved on the sheet: C48, C49, C50, C51, C52, R29, TP6, TP7, TP8, TP9, U7, VR1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
