File: Hardware/BTL_ESD/tft.kicad_sch (KiCad schematic)
At the start: 0 parts

Commit message: hardware: ver 1 schematic
Parts:
- added C42: 10uF/16V, Capacitor_SMD:C_0603_1608Metric_Pad1.08x0.95mm_HandSolder, symbol Device:C_Small
- added C43: 100nF/16V, Capacitor_SMD:C_0603_1608Metric_Pad1.08x0.95mm_HandSolder, symbol Device:C_Small
- added J3: Socket_TFT_1, XH_2_54:au_XH_2.54mm_8_Chan_Dan_SMD_Nam_Ngang, symbol Connector:Conn_01x08_Socket
- added J4: Socket_TFT_2, XH_2_54:au_XH_2.54mm_6_Chan_Dan_SMD_Nam_Ngang, symbol Connector:Conn_01x06_Socket
- added Q1: MMBT2222A, MMBT2222A:SOT103P240X110-3N, symbol MMBT2222A:MMBT2222A
- added R18: 1k/1%, Resistor_SMD:R_0603_1608Metric_Pad0.98x0.95mm_HandSolder, symbol Device:R_US
Connections:
- new net: Q1.1, R18.2
- new net +3V3: J3.8 (Pin_8), Q1.3
- new net +5V: C42.1, C43.1, J3.1 (Pin_1)
- new net GND: C42.2, C43.2, J3.2 (Pin_2), Q1.2
- new net SPI1_CS: J3.3 (Pin_3)
- new net SPI1_MISO: J4.1 (Pin_1)
- new net SPI1_MOSI: J3.6 (Pin_6)
- new net SPI1_SCLK: J3.7 (Pin_7)
- new net SPI2_CS: J4.3 (Pin_3)
- new net SPI2_MISO: J4.5 (Pin_5)
- new net SPI2_MOSI: J4.4 (Pin_4)
- new net SPI2_SCLK: J4.2 (Pin_2)
- new net TFT_BL: R18.1
- new net TFT_DC_RS: J3.5 (Pin_5)
- new net TFT_IRQ: J4.6 (Pin_6)
- new net TFT_RESET: J3.4 (Pin_4)
Other:
- title: (none) -> ILI9341

Commit message: update
Parts:
- added R31: 10k/1%, Resistor_SMD:R_0603_1608Metric_Pad0.98x0.95mm_HandSolder, symbol Device:R_US
Connections:
- net +3V3: now also R31.1; no longer J3.8 (Pin_8), Q1.3
- new net CONTROL_BL: J3.8 (Pin_8), Q1.3, R31.2
Changed lines of the file:
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@@
     (date "2024-03-08")
   )
+  (junction (at 88.9 67.31) (diameter 0) (color 0 0 0 0)
+  )
   (junction (at 132.08 63.5) (diameter 0) (color 0 0 0 0)
   )
@@
   (junction (at 116.84 63.5) (diameter 0) (color 0 0 0 0)
   )
-  (junction (at 88.9 67.31) (diameter 0) (color 0 0 0 0)
-  )
   (wire (pts (xy 146.05 69.85) (xy 146.05 73.66))
     (stroke (width 0) (type default))
@@
     (stroke (width 0) (type default))
   )
+  (wire (pts (xy 88.9 53.34) (xy 88.9 55.88))
+    (stroke (width 0) (type default))
+  )
   (wire (pts (xy 209.55 74.93) (xy 214.63 74.93))
     (stroke (width 0) (type default))
@@
     (stroke (width 0) (type default))
   )
+  (wire (pts (xy 88.9 63.5) (xy 88.9 67.31))
+    (stroke (width 0) (type default))
+  )
   (wire (pts (xy 67.31 73.66) (xy 71.12 73.66))
     (stroke (width 0) (type default))
@@
   )
   (wire (pts (xy 208.28 67.31) (xy 214.63 67.31))
-    (stroke (width 0) (type default))
-  )
-  (wire (pts (xy 88.9 62.23) (xy 88.9 67.31))
     (stroke (width 0) (type default))
   )
@@
     )
   )
+  (symbol (lib_id "Device:R_US") (at 88.9 59.69 0) (unit 1)
+    (in_bom yes) (on_board yes) (dnp no) (fields_autoplaced)
+    (property "Reference" "R31" (at 91.44 58.42 0)
+      (effects (font (size 1.27 1.27)) (justify left))
+    )
+    (property "Value" "10k/1%" (at 91.44 60.96 0)
+      (effects (font (size 1.27 1.27)) (justify left))
+    )
+    (property "Footprint" "Resistor_SMD:R_0603_1608Metric_Pad0.98x0.95mm_HandSolder" (at 89.916 59.944 90)
+      (effects (font (size 1.27 1.27)) hide)
+    )
+    (property "Datasheet" "~" (at 88.9 59.69 0)
+      (effects (font (size 1.27 1.27)) hide)
+    )
+    (property "URL" "https://www.thegioiic.com/dien-tro-10-kohm-0603-1-" (at 88.9 59.69 0)
+      (effects (font (size 1.27 1.27)) hide)
+    )
+    (pin "1")
+    (pin "2")
+    (instances
+      (project "BTL_ESD"
+        (path "/ce4779b4-6d78-42e3-84df-0a4e77629b0f/06edfd9a-10e3-4294-8775-983c56efee5c"
+          (reference "R31") (unit 1)
+        )
+      )
+    )
+  )
   (symbol (lib_id "MMBT2222A:MMBT2222A") (at 85.09 73.66 0) (unit 1)
     (in_bom yes) (on_board yes) (dnp no) (fields_autoplaced)
@@
     )
   )
-  (symbol (lib_id "power:+3V3") (at 88.9 62.23 0) (unit 1)
-    (in_bom yes) (on_board yes) (dnp no) (fields_autoplaced)
-    (property "Reference" "#PWR050" (at 88.9 66.04 0)
-      (effects (font (size 1.27 1.27)) hide)
-    )
-    (property "Value" "+3V3" (at 88.9 57.15 0)
-      (effects (font (size 1.27 1.27)))
-    )
-    (property "Footprint" "" (at 88.9 62.23 0)
-      (effects (font (size 1.27 1.27)) hide)
-    )
-    (property "Datasheet" "" (at 88.9 62.23 0)
-      (effects (font (size 1.27 1.27)) hide)
-    )
+  (symbol (lib_id "power:+3V3") (at 88.9 53.34 0) (unit 1)
+    (in_bom yes) (on_board yes) (dnp no) (fields_autoplaced)
+    (property "Reference" "#PWR050" (at 88.9 57.15 0)
+      (effects (font (size 1.27 1.27)) hide)
+    )
+    (property "Value" "+3V3" (at 88.9 48.26 0)
+      (effects (font (size 1.27 1.27)))
+    )
+    (property "Footprint" "" (at 88.9 53.34 0)
+      (effects (font (size 1.27 1.27)) hide)
+    )
+    (property "Datasheet" "" (at 88.9 53.34 0)
+      (effects (font (size 1.27 1.27)) hide)
+    )

Commit message: update
Parts:
- renumbered R31 to R19
Connections:
- net +5V: now also J3.7 (Pin_7); no longer J3.1 (Pin_1)
- net CONTROL_BL: now also J3.1 (Pin_1); no longer J3.8 (Pin_8)
- net GND: now also J3.8 (Pin_8); no longer J3.2 (Pin_2)
- net SPI1_CS: now also J3.6 (Pin_6); no longer J3.3 (Pin_3)
- net SPI1_MISO: now also J4.6 (Pin_6); no longer J4.1 (Pin_1)
- net SPI1_MOSI: now also J3.3 (Pin_3); no longer J3.6 (Pin_6)
- net SPI1_SCLK: now also J3.2 (Pin_2); no longer J3.7 (Pin_7)
- net SPI2_CS: now also J4.4 (Pin_4); no longer J4.3 (Pin_3)
- net SPI2_MISO: now also J4.2 (Pin_2); no longer J4.5 (Pin_5)
- net SPI2_MOSI: now also J4.3 (Pin_3); no longer J4.4 (Pin_4)
- net SPI2_SCLK: now also J4.5 (Pin_5); no longer J4.2 (Pin_2)
- net TFT_DC_RS: now also J3.4 (Pin_4); no longer J3.5 (Pin_5)
- net TFT_IRQ: now also J4.1 (Pin_1); no longer J4.6 (Pin_6)
- net TFT_RESET: now also J3.5 (Pin_5); no longer J3.4 (Pin_4)

Commit message: fea:STM32: upload structure fodler
Parts:
- renumbered J3 to J4, J4 to J5, R18 to R19, R19 to R20
Changed lines of the file:
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@@
   (symbol (lib_id "Connector:Conn_01x08_Socket") (at 173.99 74.93 0) (unit 1)
     (in_bom yes) (on_board yes) (dnp no) (fields_autoplaced)
-    (property "Reference" "J3" (at 175.26 74.93 0)
+    (property "Reference" "J4" (at 175.26 74.93 0)
       (effects (font (size 1.27 1.27)) (justify left))
     )
@@
       (project "BTL_ESD"
         (path "/ce4779b4-6d78-42e3-84df-0a4e77629b0f/06edfd9a-10e3-4294-8775-983c56efee5c"
-          (reference "J3") (unit 1)
+          (reference "J4") (unit 1)
         )
       )
@@
   (symbol (lib_id "Device:R_US") (at 74.93 73.66 90) (unit 1)
     (in_bom yes) (on_board yes) (dnp no) (fields_autoplaced)
-    (property "Reference" "R18" (at 74.93 67.31 90)
+    (property "Reference" "R19" (at 74.93 67.31 90)
       (effects (font (size 1.27 1.27)))
     )
@@
       (project "BTL_ESD"
         (path "/ce4779b4-6d78-42e3-84df-0a4e77629b0f/06edfd9a-10e3-4294-8775-983c56efee5c"
-          (reference "R18") (unit 1)
+          (reference "R19") (unit 1)
         )
       )
@@
   (symbol (lib_id "Device:R_US") (at 88.9 59.69 0) (unit 1)
     (in_bom yes) (on_board yes) (dnp no) (fields_autoplaced)
-    (property "Reference" "R19" (at 91.44 58.42 0)
+    (property "Reference" "R20" (at 91.44 58.42 0)
       (effects (font (size 1.27 1.27)) (justify left))
     )
@@
       (project "BTL_ESD"
         (path "/ce4779b4-6d78-42e3-84df-0a4e77629b0f/06edfd9a-10e3-4294-8775-983c56efee5c"
-          (reference "R19") (unit 1)
+          (reference "R20") (unit 1)
         )
       )
@@
   (symbol (lib_id "Connector:Conn_01x06_Socket") (at 219.71 72.39 0) (unit 1)
     (in_bom yes) (on_board yes) (dnp no) (fields_autoplaced)
-    (property "Reference" "J4" (at 220.98 72.39 0)
+    (property "Reference" "J5" (at 220.98 72.39 0)
       (effects (font (size 1.27 1.27)) (justify left))
     )
@@
       (project "BTL_ESD"
         (path "/ce4779b4-6d78-42e3-84df-0a4e77629b0f/06edfd9a-10e3-4294-8775-983c56efee5c"
-          (reference "J4") (unit 1)
-        )
-      )
+          (reference "J5") (unit 1)
+        )
+      )

Commit message: code:ESP32: update uart driver, main.c && hardware file pcb
Parts:
- renumbered R19 to R22, R20 to R23
Changed lines of the file:
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@@
   (symbol (lib_id "Device:R_US") (at 74.93 73.66 90) (unit 1)
     (in_bom yes) (on_board yes) (dnp no) (fields_autoplaced)
-    (property "Reference" "R19" (at 74.93 67.31 90)
+    (property "Reference" "R22" (at 74.93 67.31 90)
       (effects (font (size 1.27 1.27)))
     )
@@
       (project "BTL_ESD"
         (path "/ce4779b4-6d78-42e3-84df-0a4e77629b0f/06edfd9a-10e3-4294-8775-983c56efee5c"
-          (reference "R19") (unit 1)
+          (reference "R22") (unit 1)
         )
       )
@@
   (symbol (lib_id "power:GND") (at 88.9 85.09 0) (unit 1)
     (in_bom yes) (on_board yes) (dnp no) (fields_autoplaced)
-    (property "Reference" "#PWR055" (at 88.9 91.44 0)
+    (property "Reference" "#PWR056" (at 88.9 91.44 0)
       (effects (font (size 1.27 1.27)) hide)
     )
@@
       (project "BTL_ESD"
         (path "/ce4779b4-6d78-42e3-84df-0a4e77629b0f/06edfd9a-10e3-4294-8775-983c56efee5c"
-          (reference "#PWR055") (unit 1)
+          (reference "#PWR056") (unit 1)
         )
       )
@@
   (symbol (lib_id "Device:R_US") (at 88.9 59.69 0) (unit 1)
     (in_bom yes) (on_board yes) (dnp no) (fields_autoplaced)
-    (property "Reference" "R20" (at 91.44 58.42 0)
+    (property "Reference" "R23" (at 91.44 58.42 0)
       (effects (font (size 1.27 1.27)) (justify left))
     )
@@
       (project "BTL_ESD"
         (path "/ce4779b4-6d78-42e3-84df-0a4e77629b0f/06edfd9a-10e3-4294-8775-983c56efee5c"
-          (reference "R20") (unit 1)
+          (reference "R23") (unit 1)
         )
       )
@@
   (symbol (lib_id "power:+5V") (at 116.84 80.01 0) (unit 1)
     (in_bom yes) (on_board yes) (dnp no) (fields_autoplaced)
-    (property "Reference" "#PWR056" (at 116.84 83.82 0)
+    (property "Reference" "#PWR057" (at 116.84 83.82 0)
       (effects (font (size 1.27 1.27)) hide)
     )
@@
       (project "BTL_ESD"
         (path "/ce4779b4-6d78-42e3-84df-0a4e77629b0f/06edfd9a-10e3-4294-8775-983c56efee5c"
-          (reference "#PWR056") (unit 1)
+          (reference "#PWR057") (unit 1)
         )
       )
@@
   (symbol (lib_id "power:GND") (at 116.84 95.25 0) (unit 1)
     (in_bom yes) (on_board yes) (dnp no) (fields_autoplaced)
-    (property "Reference" "#PWR057" (at 116.84 101.6 0)
+    (property "Reference" "#PWR058" (at 116.84 101.6 0)
       (effects (font (size 1.27 1.27)) hide)
     )
@@
       (project "BTL_ESD"
         (path "/ce4779b4-6d78-42e3-84df-0a4e77629b0f/06edfd9a-10e3-4294-8775-983c56efee5c"
-          (reference "#PWR057") (unit 1)
+          (reference "#PWR058") (unit 1)
         )
       )
@@
   (symbol (lib_id "power:+3V3") (at 88.9 53.34 0) (unit 1)
     (in_bom yes) (on_board yes) (dnp no) (fields_autoplaced)
-    (property "Reference" "#PWR054" (at 88.9 57.15 0)
+    (property "Reference" "#PWR055" (at 88.9 57.15 0)
       (effects (font (size 1.27 1.27)) hide)
     )
@@
       (project "BTL_ESD"
         (path "/ce4779b4-6d78-42e3-84df-0a4e77629b0f/06edfd9a-10e3-4294-8775-983c56efee5c"
-          (reference "#PWR054") (unit 1)
+          (reference "#PWR055") (unit 1)
         )
       )
