File: Hardware/BTL_ESD/tft.kicad_sch (KiCad schematic)
At the start: 7 parts, among them J4 Socket_TFT_1, J5 Socket_TFT_2, Q1 MMBT2222A

Commit message: update hardware
Other:
- note added: "CONTROL BACKLIGHT"
- note added: "DISPLAY"
- note added: "TOUCH"
- moved on the sheet: J5, Q1, R22, R23
