File: Hardware/BTL_ESD/control_led.kicad_sch (KiCad schematic)
At the start: 9 parts, among them K1 SRA-05VDC-CL, Q4 MMBT2222A, U9 PC817X2NIPW

Commit message: update hardware
Other:
- note added: "CONTROL RELAY"
- note added: "ISOLATION"
Changed lines of the file:
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@@
+		)
+	)
+	(rectangle
+		(start 121.92 72.39)
+		(end 237.49 130.81)
+		(stroke
+			(width 0)
+			(type dash)
+		)
+		(fill
+			(type none)
+		)
+	)
+	(rectangle
+		(start 68.58 72.39)
+		(end 119.38 130.81)
+		(stroke
+			(width 0)
+			(type dash)
+		)
+		(fill
+			(type none)
+		)
+	)
+	(text "ISOLATION"
+		(exclude_from_sim no)
+		(at 87.376 75.184 0)
+		(effects
+			(font
+				(size 1.27 1.27)
+				(thickness 0.254)
+				(bold yes)
+			)
+			(justify left bottom)
+		)
+	)
+	(text "CONTROL RELAY"
+		(exclude_from_sim no)
+		(at 171.196 75.184 0)
+		(effects
+			(font
+				(size 1.27 1.27)
+				(thickness 0.254)
+				(bold yes)
+			)
+			(justify left bottom)
 		)
 	)
