File: Hardware/BTL_ESD/current_supply.kicad_sch (KiCad schematic)
At the start: 10 parts, among them U6 MCP6002-E_SN

Commit message: update hardware
Other:
- note added: "CURRENT POWER"
- note added: "FILTER"
- moved on the sheet: C44, C45, C46, C47
