File: Hardware/BTL_ESD/power_supply.kicad_sch (KiCad schematic)
At the start: 49 parts, among them J1 DC-005-5A-2.0, SW1 MS-22D18G2ROHS, U1 ICL7662CBA-T, U2 AMS1117-3.3, U3 TPS54331D

Commit message: update hardware
Parts:
- C13: value 1nF/50V -> 4.7nF/50V; URL https://www.thegioiic.com/tu-gom-0603-1nf-50v -> https://www.thegioiic.com/tu-gom-0603-4-7nf-50v
- C14: value 47pF/50V -> 39pF/50V; URL https://www.thegioiic.com/tu-gom-0603-47pf-50v -> https://www.thegioiic.com/tu-gom-0603-39pf-50v
- C15, C16: value 47uF/6.3V -> 33uF/6.3V
Other:
- moved on the sheet: H1, H2, H3, TP1, TP2, TP3, TP4, TP5
